Commit message: Исправлена структура проекта, чтобы он запускался

File: rc5_description/urdf/RC_5_PS.urdf (robot description, URDF)
Before this commit: robot RC 5 PS, 7 links, 6 joints
Links:
- link base_link: geometry collision mesh filename=package://rc5_description/meshes/base_link.stl; visual mesh filename=package://rc5_description/meshes/base_link.stl
- link link0: geometry collision mesh filename=package://rc5_description/meshes/link0.stl; visual mesh filename=package://rc5_description/meshes/link0.stl
- link link1: geometry collision mesh filename=package://rc5_description/meshes/link1.stl; visual mesh filename=package://rc5_description/meshes/link1.stl
- link link2: geometry collision mesh filename=package://rc5_description/meshes/link2.stl; visual mesh filename=package://rc5_description/meshes/link2.stl
- link link3: geometry collision mesh filename=package://rc5_description/meshes/link3.stl; visual mesh filename=package://rc5_description/meshes/link3.stl
- link link4: geometry collision mesh filename=package://rc5_description/meshes/link4.stl; visual mesh filename=package://rc5_description/meshes/link4.stl
- link link5: geometry collision mesh filename=package://rc5_description/meshes/link5.stl; visual mesh filename=package://rc5_description/meshes/link5.stl
